File: simple-audio-out.kicad_sch (KiCad schematic)
At the start: 10 parts, among them J1 Conn_01x04, Q1 2N3904

Commit message: #1 -- change the footprint of Q1 for easier assembly
Parts:
- Q1: footprint Package_TO_SOT_THT:TO-92_Inline -> Package_TO_SOT_THT:TO-92_Inline_Wide
Changed lines of the file:
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@@
       (effects (font (size 1.27 1.27)) (justify left))
     )
-    (property "Footprint" "Package_TO_SOT_THT:TO-92_Inline" (at 106.68 57.785 0)
+    (property "Footprint" "Package_TO_SOT_THT:TO-92_Inline_Wide" (at 106.68 57.785 0)
       (effects (font (size 1.27 1.27) italic) (justify left) hide)
     )

Commit message: #1 -- adjust the mounting holes for the speaker
Parts:
- H1, H3: footprint MountingHole:MountingHole_3.5mm -> holes:MountingHole_3.5mm_room_1.5mm
Changed lines of the file:
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@@
       (effects (font (size 1.27 1.27)))
     )
-    (property "Footprint" "MountingHole:MountingHole_3.5mm" (at 171.45 96.52 0)
+    (property "Footprint" "holes:MountingHole_3.5mm_room_1.5mm" (at 171.45 96.52 0)
       (effects (font (size 1.27 1.27)) hide)
     )
@@
       (effects (font (size 1.27 1.27)))
     )
-    (property "Footprint" "MountingHole:MountingHole_3.5mm" (at 171.45 83.82 0)
+    (property "Footprint" "holes:MountingHole_3.5mm_room_1.5mm" (at 171.45 83.82 0)
       (effects (font (size 1.27 1.27)) hide)
     )
